Commit message: debug

File: panda7/urdf/panda7.urdf (robot description, URDF)
Before this commit: robot robot, 22 links, 21 joints
Links:
- link base: geometry collision box size=0.49 0.32 0.235; visual mesh filename=../meshes/trunk.dae scale=1 1 1

File: src/robots/panda7_description/urdf/panda7.urdf (robot description, URDF)
Before this commit: robot robot, 23 links, 22 joints
Links:
- removed link head_up_realsense_link_2
- removed link imu_link
Joints:
- removed joint head_up_realsense_joint_2
- removed joint imu_joint

File: src/robots/panda7_description/xacro/gazebo.xacro (robot description, xacro)
@@ -40,5 +40,5 @@
         </plugin>
     </gazebo>
-    <gazebo reference="imu_link">
+    <gazebo reference="base">
         <gravity>true</gravity>
         <sensor name="imu_sensor" type="imu">
@@ -54,5 +54,5 @@
                 <xyzOffset>0 0 0</xyzOffset>
                 <rpyOffset>0 0 0</rpyOffset>
-                <frameName>imu_link</frameName>
+                <frameName>base</frameName>
             </plugin>
             <pose>0 0 0 0 0 0</pose>
@@ -127,108 +127,104 @@
     </xacro:if>
     <gazebo reference="base">
-        <mu1>0.2</mu1>
-        <mu2>0.2</mu2>
-        <kp  value="10000.0"/>
-        <kd  value="1.0"/>
-    </gazebo>
-    <gazebo reference="imu_link">
-        <mu1>0.2</mu1>
-        <mu2>0.2</mu2>
+        <mu1>0.6</mu1>
+        <mu2>0.6</mu2>
+        <kp  value="100000.0"/>
+        <kd  value="10.0"/>
     </gazebo>
     <!-- FL leg -->
     <gazebo reference="FL_hip">
-        <mu1>0.2</mu1>
-        <mu2>0.2</mu2>
+        <mu1>0.6</mu1>
+        <mu2>0.6</mu2>
     </gazebo>
     <gazebo reference="FL_thigh">
-        <mu1>0.2</mu1>
-        <mu2>0.2</mu2>
-        <self_collide>1</self_collide>
-        <kp  value="10000.0"/>
-        <kd  value="1.0"/>
+        <mu1>0.6</mu1>
+        <mu2>0.6</mu2>
+        <self_collide>0</self_collide>
+        <kp value="200000.0"/>   <!-- 2e5 -->
+        <kd value="20.0"/>
     </gazebo>
     <gazebo reference="FL_calf">
-        <mu1>0.2</mu1>
-        <mu2>0.2</mu2>
-        <self_collide>1</self_collide>
+        <mu1>0.8</mu1>
+        <mu2>0.8</mu2>
+        <self_collide>0</self_collide>
     </gazebo>
     <gazebo reference="FL_foot">
-        <mu1>0.6</mu1>
-        <mu2>0.6</mu2>
-        <self_collide>1</self_collide>
-        <kp  value="10000.0"/>
-        <kd  value="1.0"/>
+         <mu1>1.0</mu1>
+        <mu2>1.0</mu2>
+        <self_collide>0</self_collide>
+        <kp  value="200000.0"/>
+        <kd  value="20.0"/>
     </gazebo>
     <!-- FR leg -->
     <gazebo reference="FR_hip">
-        <mu1>0.2</mu1>
-        <mu2>0.2</mu2>
+        <mu1>0.6</mu1>
+        <mu2>0.6</mu2>
     </gazebo>
     <gazebo reference="FR_thigh">
-        <mu1>0.2</mu1>
-        <mu2>0.2</mu2>
-        <self_collide>1</self_collide>
-        <kp  value="10000.0"/>
-        <kd  value="1.0"/>
+        <mu1>0.6</mu1>
+        <mu2>0.6</mu2>
+        <self_collide>0</self_collide>
+        <kp value="200000.0"/>   <!-- 2e5 -->
+        <kd value="20.0"/>
     </gazebo>
     <gazebo reference="FR_calf">
-        <mu1>0.2</mu1>
-        <mu2>0.2</mu2>
-        <self_collide>1</self_collide>
+        <mu1>0.8</mu1>
+        <mu2>0.8</mu2>
+        <self_collide>0</self_collide>
     </gazebo>
     <gazebo reference="FR_foot">
-        <mu1>0.6</mu1>
-        <mu2>0.6</mu2>
-        <self_collide>1</self_collide>
-        <kp  value="10000.0"/>
-        <kd  value="1.0"/>
+        <mu1>1.0</mu1>
+        <mu2>1.0</mu2>
+        <self_collide>0</self_collide>
+        <kp  value="200000.0"/>
+        <kd  value="20.0"/>
     </gazebo>
     <!-- RL leg -->
     <gazebo reference="RL_hip">
-        <mu1>0.2</mu1>
-        <mu2>0.2</mu2>
+        <mu1>0.6</mu1>
+        <mu2>0.6</mu2>
     </gazebo>
     <gazebo reference="RL_thigh">
-        <mu1>0.2</mu1>
-        <mu2>0.2</mu2>
-        <self_collide>1</self_collide>
-        <kp  value="10000.0"/>
-        <kd  value="1.0"/>
+        <mu1>0.6</mu1>
+        <mu2>0.6</mu2>
+        <self_collide>0</self_collide>
+        <kp value="200000.0"/>   <!-- 2e5 -->
+        <kd value="20.0"/>
     </gazebo>
     <gazebo reference="RL_calf">
-        <mu1>0.2</mu1>
-        <mu2>0.2</mu2>
-        <self_collide>1</self_collide>
+        <mu1>0.8</mu1>
+        <mu2>0.8</mu2>
+        <self_collide>0</self_collide>
     </gazebo>
     <gazebo reference="RL_foot">
-        <mu1>0.6</mu1>
-        <mu2>0.6</mu2>
-        <self_collide>1</self_collide>
-        <kp  value="10000.0"/>
-        <kd  value="1.0"/>
+        <mu1>1.0</mu1>
+        <mu2>1.0</mu2>
+        <self_collide>0</self_collide>
+        <kp  value="200000.0"/>
+        <kd  value="20.0"/>
     </gazebo>
     <!-- RR leg -->
     <gazebo reference="RR_hip">
-        <mu1>0.2</mu1>
-        <mu2>0.2</mu2>
+        <mu1>0.6</mu1>
+        <mu2>0.6</mu2>
     </gazebo>
     <gazebo reference="RR_thigh">
-        <mu1>0.2</mu1>
-        <mu2>0.2</mu2>
-        <self_collide>1</self_collide>
-        <kp  value="10000.0"/>
-        <kd  value="1.0"/>
+        <mu1>0.6</mu1>
+        <mu2>0.6</mu2>
+        <self_collide>0</self_collide>
+        <kp value="200000.0"/>   <!-- 2e5 -->
+        <kd value="20.0"/>
     </gazebo>
     <gazebo reference="RR_calf">
-        <mu1>0.2</mu1>
-        <mu2>0.2</mu2>
-        <self_collide>1</self_collide>
+        <mu1>0.8</mu1>
+        <mu2>0.8</mu2>
+        <self_collide>0</self_collide>
     </gazebo>
     <gazebo reference="RR_foot">
-        <mu1>0.6</mu1>
-        <mu2>0.6</mu2>
-        <self_collide>1</self_collide>
-        <kp  value="10000.0"/>
-        <kd  value="1.0"/>
+        <mu1>1.0</mu1>
+        <mu2>1.0</mu2>
+        <self_collide>0</self_collide>
+        <kp  value="200000.0"/>
+        <kd  value="20.0"/>
     </gazebo>
 </robot>
