Commit message: add crouch model

File: rl_sar/src/rl_sar_zoo/panda3_description/urdf/panda3.backup.urdf (robot description, URDF)
Before this commit: robot MCat, 17 links, 16 joints
Links:
- added link imu_link, mass 0
- link FL_calf: geometry collision box size=0.22 0.02 0.0495; collision cylinder length=0.02 radius=0.013
- link FL_foot: geometry collision sphere radius=0.027; visual mesh filename=package://panda3_description/meshes/FL_foot.STL
- link FL_thigh: geometry collision box size=0.050 0.03 0.21; collision cylinder length=0.129 radius=0.05
- link FR_calf: geometry collision box size=0.22 0.02 0.0495; collision cylinder length=0.02 radius=0.013
- link FR_foot: geometry collision sphere radius=0.027; visual mesh filename=package://panda3_description/meshes/FR_foot.STL
- link FR_thigh: geometry collision box size=0.050 0.03 0.21; collision cylinder length=0.129 radius=0.05
- link RL_calf: geometry collision box size=0.22 0.02 0.0495; collision cylinder length=0.02 radius=0.013
- link RL_foot: geometry collision sphere radius=0.027; visual mesh filename=package://panda3_description/meshes/RL_foot.STL
- link RL_thigh: geometry collision box size=0.050 0.03 0.21; collision cylinder length=0.129 radius=0.05
- link RR_calf: geometry collision box size=0.22 0.02 0.0495; collision cylinder length=0.02 radius=0.013
- link RR_foot: geometry collision sphere radius=0.027; visual mesh filename=package://panda3_description/meshes/RR_foot.STL
- link RR_thigh: geometry collision box size=0.050 0.03 0.21; collision cylinder length=0.129 radius=0.05
- link base: geometry collision box size=0.03 0.17 0.110; collision box size=0.03 0.18 0.120
Joints:
- added joint imu_joint: type fixed, parent base, child imu_link, origin xyz=0 0 0 rpy=0 0 0, axis 0 0 0
- joint FL_calf_joint: limit lower=-2.443 upper=0.524 effort=90 velocity=19.9 -> lower=-2.53 upper=0.35 effort=90 velocity=19.9
- joint FL_thigh_joint: limit lower=-1.62 upper=3.735 effort=60 velocity=19.9 -> lower=-1.571 upper=3.75 effort=60 velocity=19.9
- joint FR_calf_joint: limit lower=-2.44 upper=0.52 effort=90 velocity=19.9 -> lower=-2.53 upper=0.35 effort=90 velocity=19.9
- joint FR_thigh_joint: limit lower=-1.62 upper=3.73 effort=60 velocity=19.9 -> lower=-1.57 upper=3.75 effort=60 velocity=19.9
- joint RL_calf_joint: limit lower=-2.44 upper=0.52 effort=90 velocity=19.9 -> lower=-2.53 upper=0.35 effort=90 velocity=19.9
- joint RL_thigh_joint: limit lower=-1.62 upper=3.73 effort=60 velocity=19.9 -> lower=-1.57 upper=3.75 effort=60 velocity=19.9
- joint RR_calf_joint: limit lower=-2.44 upper=0.52 effort=90 velocity=19.9 -> lower=-2.53 upper=0.35 effort=90 velocity=19.9
- joint RR_thigh_joint: limit lower=-1.62 upper=3.73 effort=4.8 velocity=19.9 -> lower=-1.57 upper=3.752 effort=4.8 velocity=19.9
