Commit message: 恢复

File: rl_sar/src/rl_sar_zoo/panda3_description/urdf/panda3.urdf (robot description, URDF)
Before this commit: robot MCat, 17 links, 16 joints
Links:
- link FL_calf: mass 0.8806081 -> 0.22017362; geometry collision box size=0.2 0.02 0.035; visual mesh filename=package://panda3_description/meshes/FL_calf.STL
- link FL_foot: mass 0.0333176 -> 0.03331764
- link FL_hip: mass 1.2535095 -> 1.12888829; geometry visual mesh filename=package://panda3_description/meshes/FL_hip.STL
- link FL_thigh: mass 1.6830194 -> 1.96466711; geometry collision box size=0.044 0.03 0.16; collision cylinder length=0.12 radius=0.05
- link FR_calf: mass 0.8709683 -> 0.22016958; geometry collision box size=0.2 0.02 0.035; visual mesh filename=package://panda3_description/meshes/FR_calf.STL
- link FR_foot: mass 0.0333176 -> 0.03331764
- link FR_hip: mass 1.2535095 -> 1.12888829; geometry visual mesh filename=package://panda3_description/meshes/FR_hip.STL
- link FR_thigh: mass 1.6556826 -> 1.96467358; geometry collision box size=0.044 0.03 0.16; collision cylinder length=0.12 radius=0.05
- link RL_calf: mass 0.8806081 -> 0.22017362; geometry collision box size=0.2 0.02 0.035; visual mesh filename=package://panda3_description/meshes/RL_calf.STL
- link RL_foot: mass 0.0333176 -> 0.03331764
- link RL_hip: mass 1.2535095 -> 1.12888829; geometry visual mesh filename=package://panda3_description/meshes/RL_hip.STL
- link RL_thigh: mass 1.6830194 -> 1.96466711; geometry collision box size=0.044 0.03 0.16; collision cylinder length=0.12 radius=0.05
- link RR_calf: mass 0.8709683 -> 0.22016958; geometry collision box size=0.2 0.02 0.035; visual mesh filename=package://panda3_description/meshes/RR_calf.STL
- link RR_foot: mass 0.0333176 -> 0.03331764
- link RR_hip: mass 1.2535095 -> 1.12888829; geometry visual mesh filename=package://panda3_description/meshes/RR_hip.STL
- link RR_thigh: mass 1.6556826 -> 1.96467358; geometry collision box size=0.044 0.03 0.16; collision cylinder length=0.12 radius=0.05
- link base: mass 15.2817858 -> 20.90069011; geometry collision box size=0.32 0.16 0.16; collision cylinder length=0.32 radius=0.08
Joints:
- joint FL_calf_joint: limit lower=-2.443 upper=0.524 effort=90 velocity=19.9 -> lower=-2.443 upper=-0.524 effort=90 velocity=14.0
- joint FL_hip_joint: limit lower=-1.047 upper=1.047 effort=60 velocity=19.9 -> lower=-0.8 upper=0.8 effort=60 velocity=14.0; origin xyz=0.28494 0.079803 -0.015554 rpy=0 0 0 -> xyz=0.286 0.082 -0.0 rpy=0 0 0
- joint FL_thigh_joint: limit lower=-1.62 upper=3.735 effort=60 velocity=19.9 -> lower=-1.62 upper=3.735 effort=60 velocity=14.0
- joint FR_calf_joint: limit lower=-2.44 upper=0.52 effort=90 velocity=19.9 -> lower=-2.44 upper=-0.52 effort=90 velocity=14.0
- joint FR_hip_joint: limit lower=-1.047 upper=1.047 effort=60 velocity=19.9 -> lower=-0.8 upper=0.8 effort=60 velocity=14.0; origin xyz=0.28494 -0.084197 -0.015554 rpy=0 0 0 -> xyz=0.286 -0.082 -0.0 rpy=0 0 0
- joint FR_thigh_joint: limit lower=-1.62 upper=3.73 effort=60 velocity=19.9 -> lower=-1.62 upper=3.73 effort=60 velocity=14.0
- joint RL_calf_joint: limit lower=-2.44 upper=0.52 effort=90 velocity=19.9 -> lower=-2.44 upper=-0.52 effort=90 velocity=14.0
- joint RL_hip_joint: limit lower=-1.047 upper=1.047 effort=60 velocity=19.9 -> lower=-0.8 upper=0.8 effort=60 velocity=14.0; origin xyz=-0.28906 0.079803 -0.015554 rpy=0 0 0 -> xyz=-0.286 0.082 -0.0 rpy=0 0 0
- joint RL_thigh_joint: limit lower=-1.62 upper=3.73 effort=60 velocity=19.9 -> lower=-1.62 upper=3.73 effort=60 velocity=14.0
- joint RR_calf_joint: limit lower=-2.44 upper=0.52 effort=90 velocity=19.9 -> lower=-2.44 upper=-0.52 effort=90 velocity=14.0
- joint RR_hip_joint: limit lower=-1.047 upper=1.047 effort=60 velocity=19.9 -> lower=-0.8 upper=0.8 effort=60 velocity=14.0; origin xyz=-0.28906 -0.084197 -0.015554 rpy=0 0 0 -> xyz=-0.286 -0.082 -0.0 rpy=0 0 0
- joint RR_thigh_joint: limit lower=-1.62 upper=3.73 effort=4.8 velocity=19.9 -> lower=-1.62 upper=3.73 effort=60 velocity=14.0

File: rl_sar/src/rl_sar_zoo/panda3_description/xacro/gazebo.xacro (robot description, xacro)
@@ -50,5 +50,5 @@
                 <frameName>imu_link</frameName>
             </plugin>
-            <pose>0 0 0 0 0 0</pose>
+            <pose>0.1 0.05 0 0 0 0</pose>
         </sensor>
     </gazebo>

File: rl_sar/src/rl_sar_zoo/panda3_description/xacro/robot.xacro (robot description, xacro)
@@ -1,6 +1,6 @@
 <?xml version="1.0"?>
 <robot name="panda3_description" xmlns:xacro="http://www.ros.org/wiki/xacro">
-    <xacro:include filename="$(find panda3_description)/urdf/panda3_description.urdf"/>
-    <!-- <xacro:include filename="$(find panda3_description)/urdf/panda3.urdf"/> -->
+    <!-- <xacro:include filename="$(find panda3_description)/urdf/panda3_description.urdf"/> -->
+    <xacro:include filename="$(find panda3_description)/urdf/panda3.urdf"/>
     <!-- gazebo sim -->
     <xacro:include filename="$(find panda3_description)/xacro/gazebo.xacro"/>
