Commit message: add models

File: rl_sar/src/rl_sar_zoo/panda3_description/mjcf/panda3.urdf (robot description, URDF)
Before this commit: robot MCat, 17 links, 16 joints
Links:
- link FL_hip: geometry visual mesh filename=./FL_hip.STL

File: rl_sar/src/rl_sar_zoo/panda3_description/xacro/gazebo.xacro (robot description, xacro)
@@ -143,8 +143,8 @@
             <xacro:joint_interface joint_name="${prefix}_calf_joint" torque_limit="${calf_torque_max}"/>
         </xacro:macro>
+        <xacro:leg_joints prefix="FL"/>
         <xacro:leg_joints prefix="FR"/>
-        <xacro:leg_joints prefix="FL"/>
+        <xacro:leg_joints prefix="RL"/>
         <xacro:leg_joints prefix="RR"/>
-        <xacro:leg_joints prefix="RL"/>
     </ros2_control>
     <gazebo>

File: rl_sar/src/rl_sar_zoo/panda3_description/xacro/real.xacro (robot description, xacro)
@@ -19,8 +19,8 @@
             <xacro:joint_interface joint_name="${prefix}_calf_joint" />
         </xacro:macro>
+        <xacro:leg_joints prefix="FL"/>
         <xacro:leg_joints prefix="FR"/>
-        <xacro:leg_joints prefix="FL"/>
+        <xacro:leg_joints prefix="RL"/>
         <xacro:leg_joints prefix="RR"/>
-        <xacro:leg_joints prefix="RL"/>
     </ros2_control>
 </robot>

File: rl_sar/src/rl_sar_zoo/panda3_description/xacro/robot_real.xacro (robot description, xacro)
@@ -3,4 +3,4 @@
     <xacro:include filename="$(find panda3_description)/urdf/panda3.urdf"/>
     <!-- real robot -->
-    <xacro:include filename="$(find panda7_description)/xacro/real.xacro"/>
+    <xacro:include filename="$(find panda3_description)/xacro/real.xacro"/>
 </robot>

Commit message: 存档

File: rl_sar/src/rl_sar_zoo/panda3_description/mjcf/panda3.urdf (robot description, URDF)
Before this commit: robot MCat, 17 links, 16 joints
Links:
- link base: geometry collision box size=0.03 0.17 0.110; collision box size=0.03 0.18 0.120
Joints:
- joint FL_thigh_joint: origin xyz=0 0.1055 0 rpy=0 0 0 -> xyz=0.0 0.1055 0 rpy=0 0 0

File: rl_sar/src/rl_sar_zoo/panda3_description/xacro/gazebo.xacro (robot description, xacro)
@@ -50,5 +50,5 @@
                 <frameName>imu_link</frameName>
             </plugin>
-            <pose>0.1 0.05 0 0 0 0</pose>
+            <pose>0.0 0.0 0 0 0 0</pose>
         </sensor>
     </gazebo>
