Commit message: wmp model finish

File: rl_sar/src/rl_sar_zoo/go2_description/urdf/go2_description.urdf (robot description, URDF)
Before this commit: robot go2_description, 30 links, 29 joints
Joints:
- joint FL_calf_joint: limit lower=-2.7227 upper=-0.83776 effort=45.43 velocity=15.70 -> lower=-2.7227 upper=-0.83776 effort=40.55 velocity=20.07
- joint FR_calf_joint: limit lower=-2.7227 upper=-0.83776 effort=45.43 velocity=15.70 -> lower=-2.7227 upper=-0.83776 effort=40.55 velocity=20.07
- joint RL_calf_joint: limit lower=-2.7227 upper=-0.83776 effort=45.43 velocity=15.70 -> lower=-2.7227 upper=-0.83776 effort=40.55 velocity=20.07
- joint RR_calf_joint: limit lower=-2.7227 upper=-0.83776 effort=45.43 velocity=15.70 -> lower=-2.7227 upper=-0.83776 effort=40.55 velocity=20.07

File: rl_sar/src/rl_sar_zoo/go2_description/xacro/gazebo.xacro (robot description, xacro)
@@ -193,4 +193,39 @@
           </linear_acceleration>
         </imu>
+      </sensor>
+    </gazebo>
+    <gazebo reference="base">
+      <!-- ========== 深度相机 ========== -->
+      <sensor name="depth_camera" type="depth">
+        <always_on>true</always_on>
+        <update_rate>10</update_rate>
+        <visualize>false</visualize>
+        <!-- position = [0.37, 0, 0.03]
+             y_angle = pitch 下俯，单位弧度 -->
+        <!-- <pose>0.345 0 0.05 0 0.122 0</pose> -->
+        <!-- <pose>0.37 0 0.03 0 0.0698 0</pose> -->
+        <!-- <pose>0.37 0 0.03 0 0.0698 0</pose> -->
+        <!-- <pose>0.33 0 0.128 0 0 0</pose> -->
+        <pose>0.345 0 0.05 0 0.4538 0</pose>
+        <!-- 0.122 rad ≈ 7° -->
+        <camera>
+          <!-- 58° → 弧度 -->
+          <horizontal_fov>1.012</horizontal_fov>
+          <image>
+            <width>64</width>
+            <height>64</height>
+            <format>R32F</format>
+          </image>
+          <clip>
+            <near>0.01</near>
+            <far>3.0</far>
+          </clip>
+        </camera>
+        <plugin name="depth_camera_plugin" filename="libgazebo_ros_camera.so">
+          <ros>
+            <namespace>/depth</namespace>
+          </ros>
+          <frame_name>base</frame_name>
+        </plugin>
       </sensor>
     </gazebo>

File: rl_sar/src/rl_sar_zoo/panda3_description/xacro/gazebo.xacro (robot description, xacro)
@@ -144,9 +144,19 @@
         </imu>
       </sensor>
+      <sensor name="odometry_sensor" type="odom">
+        <plugin name="odom_plugin" filename="libgazebo_ros_p3d.so">
+          <ros>
+            <namespace>/</namespace>
+            <remapping>~/odom:=odom</remapping>
+          </ros>
+          <body_name>base</body_name>
+          <frame_name>odom</frame_name>
+          <update_rate>100.0</update_rate>
+        </plugin>
+      </sensor>
       <!-- ========== 深度相机 ========== -->
       <sensor name="depth_camera" type="depth">
         <always_on>true</always_on>
-        <!-- 建议 20Hz，1024 env 不然会爆 -->
-        <update_rate>20</update_rate>
+        <update_rate>40</update_rate>
         <visualize>false</visualize>
         <!-- position = [0.37, 0, 0.03]
@@ -154,6 +164,38 @@
         <!-- <pose>0.345 0 0.05 0 0.122 0</pose> -->
         <!-- <pose>0.37 0 0.03 0 0.0698 0</pose> -->
-        <pose>0.37 0 0.03 0 0.0698 0</pose>
-        <!-- 0.122 rad ≈ 7° -->
+        <!-- <pose>0.37 0 0.03 0 0.0698 0</pose> -->
+        <!-- <pose>0.33 0 0.128 0 0 0</pose> -->
+        <pose>0.3195 0 0.1115 0 0.174533 0</pose>
+         <!-- <pose>0.3195 0 0.1815 0 0.523599 0</pose> -->
+        <!-- 0.017453 rad ≈ 1° -->
+        <!-- 0.034907 rad ≈ 2° -->
+        <!-- 0.052360 rad ≈ 3° -->
+        <!-- 0.069813 rad ≈ 4° -->
+        <!-- 0.087266 rad ≈ 5° -->
+        <!-- 0.104720 rad ≈ 6° -->
+        <!-- 0.122173 rad ≈ 7° -->
+        <!-- 0.139626 rad ≈ 8° -->
+        <!-- 0.157080 rad ≈ 9° -->
+        <!-- 0.174533 rad ≈ 10° -->
+        <!-- 0.191986 rad ≈ 11° -->
+        <!-- 0.209440 rad ≈ 12° -->
+        <!-- 0.226893 rad ≈ 13° -->
+        <!-- 0.244346 rad ≈ 14° -->
+        <!-- 0.261799 rad ≈ 15° -->
+        <!-- 0.279253 rad ≈ 16° -->
+        <!-- 0.296706 rad ≈ 17° -->
+        <!-- 0.314159 rad ≈ 18° -->
+        <!-- 0.331613 rad ≈ 19° -->
+        <!-- 0.349066 rad ≈ 20° -->
+        <!-- 0.366519 rad ≈ 21° -->
+        <!-- 0.383972 rad ≈ 22° -->
+        <!-- 0.401426 rad ≈ 23° -->
+        <!-- 0.418879 rad ≈ 24° -->
+        <!-- 0.436332 rad ≈ 25° -->
+        <!-- 0.453786 rad ≈ 26° -->
+        <!-- 0.471239 rad ≈ 27° -->
+        <!-- 0.488692 rad ≈ 28° -->
+        <!-- 0.506145 rad ≈ 29° -->
+        <!-- 0.523599 rad ≈ 30° -->
         <camera>
           <!-- 58° → 弧度 -->
@@ -165,6 +207,6 @@
           </image>
           <clip>
-            <near>0.054</near>
-            <far>40.0</far>
+            <near>0.01</near>
+            <far>3.0</far>
           </clip>
         </camera>
